File: pcb/matrix.sch (KiCad schematic (older format))
At the start: 136 parts

Commit message: Bakeneko-70 intial implementation
Parts:
- added D64, D65, D66, D67, D68, D69, D70, D71, D72, D73, D74, D75, D76, D77: 1N4148, Diode_SMD:D_SOD-123, symbol Device:D
- added MX74, MX75, MX76, MX77, MX78, MX79, MX80, MX81, MX82, MX83, MX84, MX85, MX86, MX87: 1u, MX_Only:MXOnly-1U-NoLED, symbol Switch:SW_SPST
Connections:
- net COL0: now also MX74.2 (B)
- net COL1: now also MX75.2 (B)
- net COL10: now also MX83.2 (B)
- net COL11: now also MX84.2 (B)
- net COL12: now also MX85.2 (B)
- net COL13: now also MX86.2 (B)
- net COL14: now also MX87.2 (B)
- net COL2: now also MX76.2 (B)
- net COL3: now also MX77.2 (B)
- net COL4: now also MX78.2 (B)
- net COL6: now also MX79.2 (B)
- net COL7: now also MX80.2 (B)
- net COL8: now also MX81.2 (B)
- net COL9: now also MX82.2 (B)
- new net: D64.2 (A), MX74.1 (A)
- new net: D65.2 (A), MX75.1 (A)
- new net: D66.2 (A), MX76.1 (A)
- new net: D67.2 (A), MX77.1 (A)
- new net: D68.2 (A), MX78.1 (A)
- new net: D69.2 (A), MX79.1 (A)
- new net: D70.2 (A), MX80.1 (A)
- new net: D71.2 (A), MX81.1 (A)
- new net: D72.2 (A), MX82.1 (A)
- new net: D73.2 (A), MX83.1 (A)
- new net: D74.2 (A), MX84.1 (A)
- new net: D75.2 (A), MX85.1 (A)
- new net: D76.2 (A), MX86.1 (A)
- new net: D77.2 (A), MX87.1 (A)
- new net FROW: D64.1 (K), D65.1 (K), D66.1 (K), D67.1 (K), D68.1 (K), D69.1 (K), D70.1 (K), D71.1 (K), D72.1 (K), D73.1 (K), D74.1 (K), D75.1 (K), D76.1 (K), D77.1 (K)
Other:
- moved on the sheet: D1, D10, D11, D12, D13, D14, D15, D16, D17, D18, D19, D2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
