File: pcb/bakeneko-60-pcb.kicad_pcb (KiCad board)
At the start: 2 copper layers, 284.7 x 94.2 mm, 154 parts, among them J1 JST SH 4-pin, J2 AVR-ISP-6, SW1 Reset, U1 SRV05-4, U2 ATmega32U4-AU, Y1 16MHz

Commit message: Bakeneko-70 intial implementation
Parts:
- added D64: 1N4148, Diode_SMD:D_SOD-123, B.Cu at (7.94, -23.0)
- added D65: 1N4148, Diode_SMD:D_SOD-123, B.Cu at (14.3, -23.0)
- added D66: 1N4148, Diode_SMD:D_SOD-123, B.Cu at (33.3, -23.0)
- added D67: 1N4148, Diode_SMD:D_SOD-123, B.Cu at (52.4, -23.0)
- added D68: 1N4148, Diode_SMD:D_SOD-123, B.Cu at (71.4, -23.0)
- added D69: 1N4148, Diode_SMD:D_SOD-123, B.Cu at (95.2, -23.0)
- added D70: 1N4148, Diode_SMD:D_SOD-123, B.Cu at (114.3, -23.0)
- added D71: 1N4148, Diode_SMD:D_SOD-123, B.Cu at (133.3, -23.0)
- added D72: 1N4148, Diode_SMD:D_SOD-123, B.Cu at (152.4, -23.0)
- added D73: 1N4148, Diode_SMD:D_SOD-123, B.Cu at (176.2, -23.0)
- added D74: 1N4148, Diode_SMD:D_SOD-123, B.Cu at (195.3, -23.0)
- added D75: 1N4148, Diode_SMD:D_SOD-123, B.Cu at (214.3, -23.0)
- added D76: 1N4148, Diode_SMD:D_SOD-123, B.Cu at (233.4, -23.0)
- added D77: 1N4148, Diode_SMD:D_SOD-123, B.Cu at (257.2, -23.0)
- added G1: Signature, Ramon:Signature, B.Cu at (254.8, -14.7)
- added MX74: 1u, MX_Only:MXOnly-1U-NoLED, F.Cu at (0.00, -23.8)
- added MX75: 1u, MX_Only:MXOnly-1U-NoLED, F.Cu at (23.8, -23.8)
- added MX76: 1u, MX_Only:MXOnly-1U-NoLED, F.Cu at (42.9, -23.8)
- added MX77: 1u, MX_Only:MXOnly-1U-NoLED, F.Cu at (61.9, -23.8)
- added MX78: 1u, MX_Only:MXOnly-1U-NoLED, F.Cu at (81.0, -23.8)
- added MX79: 1u, MX_Only:MXOnly-1U-NoLED, F.Cu at (104.8, -23.8)
- added MX80: 1u, MX_Only:MXOnly-1U-NoLED, F.Cu at (123.8, -23.8)
- added MX81: 1u, MX_Only:MXOnly-1U-NoLED, F.Cu at (142.9, -23.8)
- added MX82: 1u, MX_Only:MXOnly-1U-NoLED, F.Cu at (161.9, -23.8)
- added MX83: 1u, MX_Only:MXOnly-1U-NoLED, F.Cu at (185.7, -23.8)
- added MX84: 1u, MX_Only:MXOnly-1U-NoLED, F.Cu at (204.8, -23.8)
- added MX85: 1u, MX_Only:MXOnly-1U-NoLED, F.Cu at (223.8, -23.8)
- added MX86: 1u, MX_Only:MXOnly-1U-NoLED, F.Cu at (242.9, -23.8)
- added MX87: 1u, MX_Only:MXOnly-1U-NoLED, F.Cu at (266.7, -23.8)
- moved D29 12.7 mm to (252.4, 19.8)
- moved MX4 12.7 mm to (57.1, 0.00)
- moved MX45 12.7 mm to (11.9, 57.1)
- moved MX46 12.7 mm to (42.9, 57.1)
- moved MX48 12.7 mm to (81.0, 57.1)
- moved MX49 12.7 mm to (100.0, 57.1)
- moved MX50 12.7 mm to (119.1, 57.1)
- moved MX51 12.7 mm to (138.1, 57.1)
- moved MX52 12.7 mm to (157.2, 57.1)
- moved MX53 12.7 mm to (176.2, 57.1)
- moved MX54 12.7 mm to (195.3, 57.1)
- moved MX55 12.7 mm to (214.3, 57.1)
- moved MX56 12.7 mm to (240.5, 57.1)
- moved MX57 12.7 mm to (266.7, 57.1)
- moved MX58 12.7 mm to (250.0, 57.1)
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Connections:
- U2 pad 41: Net-(U2-Pad41) -> FROW
Routing:
- net FROW: track 0.00 -> 305.0 mm, vias 0 -> 2
- net COL2: track 145.1 -> 174.2 mm
- net COL14: track 314.2 -> 342.0 mm
- net COL9: track 236.0 -> 263.8 mm
- net COL8: track 217.4 -> 245.1 mm
- net COL6: track 212.3 -> 240.1 mm
- net COL7: track 198.8 -> 226.5 mm
- net COL11: track 295.1 -> 320.9 mm
- net COL10: track 274.7 -> 300.5 mm
- net COL3: track 125.1 -> 150.9 mm
- net COL1: track 110.2 -> 136.0 mm
- net COL4: track 143.4 -> 169.2 mm
- net COL13: track 351.9 -> 377.7 mm
- net COL12: track 325.5 -> 351.2 mm
- net COL0: track 100.5 -> 124.3 mm
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Other:
- board size 284.7 x 94.2 mm -> 284.7 x 118 mm
- board text added: "Bakeneko 70 v1.0 based on the Bakeneko 60 v3.0 by kkatano"
- board text removed: "Bakeneko 60 v3.0"

Commit message: Add bakeneko 70 files
Parts:
- moved G1 40.5 mm to (214.3, -12.7)
Other:
- outline, holes or cut-outs redrawn
